Commit message: update with new charger and camera mount design

File: aubo_gazebo/urdf/aubo_i5.xacro (robot description, xacro)
@@ -337,5 +337,5 @@
   <!--////////////////////////////////CameraMount_Joint/////////////////////////////////-->
   <joint name="knife_camera_mount_joint" type="fixed">
-    <origin xyz="0.0 0.115 0.01" rpy="0.0 0.0 0.0"/>
+    <origin xyz="0.0 0.11575 0.01288" rpy="0.0 0.0 0.0"/>
     <parent link="wrist3_Link"/>
     <child link="camera_mount_link"/>
@@ -371,5 +371,5 @@
       <origin xyz="0.0 0.0 0.0" rpy="0 0 0"/>
       <geometry>
-         <mesh filename="package://aubo_description/meshes/charger.STL" />
+         <mesh filename="package://aubo_description/meshes/charger.stl" />
       </geometry>
     </collision>
@@ -387,5 +387,5 @@
   <!--////////////////////////////////knife_charger_joint/////////////////////////////////-->
   <joint name="knife_charger_joint" type="fixed">
-    <origin xyz="0.06001 -0.08415 0.04208" rpy="0.0 1.5707 0.0"/>
+    <origin xyz="0.065 -0.08975 0.060" rpy="0.0 0.0 0.0"/>
     <parent link="camera_mount_link"/>
     <child link="charger_link"/>
@@ -395,5 +395,5 @@
   <link name="ee_link"/>
   <joint name="ee_link_joint" type="fixed">
-      <origin xyz="0 -0.112 0.20667" rpy="-1.5707 0.0 0.0"/>
+      <origin xyz="0 -0.11575 0.20807" rpy="-1.5707 0.0 0.0"/>
       <parent link="camera_mount_link"/>
       <child link="ee_link" />
@@ -401,5 +401,5 @@
   <link name="charger_ee_link"/>
   <joint name="charger_ee_link_joint" type="fixed">
-      <origin xyz="0 0 0.047" rpy="0.0 -1.5707 -1.5707"/>
+      <origin xyz="0.053 0.0 0.0" rpy="${-M_PI/2} 0.0 0.0"/>
       <parent link="charger_link"/>
       <child link="charger_ee_link" />

Commit message: update with new model

File: aubo_gazebo/urdf/aubo_i5.xacro (robot description, xacro)
@@ -108,5 +108,5 @@
                   izz="0.003879257" />
     </xacro:macro>
-    <xacro:macro name="Charger_Inertia">
+    <!--xacro:macro name="Charger_Inertia">
         <origin xyz="0 0 0"
                 rpy="0 0 0"/>
@@ -118,5 +118,5 @@
                   iyz="0.0"
                   izz="0.003879257" />
-    </xacro:macro>
+    </xacro:macro-->
     <!--/////////////////////////////// BASE_LINK ////////////////////////////////////-->
    <link name="base_link">
@@ -337,5 +337,5 @@
   <!--////////////////////////////////CameraMount_Joint/////////////////////////////////-->
   <joint name="knife_camera_mount_joint" type="fixed">
-    <origin xyz="0.0 0.11575 0.01288" rpy="0.0 0.0 0.0"/>
+    <origin xyz="0.0 0.0 0.005" rpy="0.0 -1.5707 -1.5707"/>
     <parent link="wrist3_Link"/>
     <child link="camera_mount_link"/>
@@ -362,10 +362,10 @@
   <!--////////////////////////////////camera_joint/////////////////////////////////-->
   <joint name="camera_joint" type="fixed">
-    <origin xyz="0.0149 0.0 0.012" rpy="0.0 -1.5707 -1.5707"/>
+    <origin xyz="0.02175 0.0149 -0.0185" rpy="0.0 0.0 0"/>
     <parent link="camera_mount_link"/>
     <child link="camera_link"/>
   </joint>
   <!--////////////////////////////////charger/////////////////////////////////-->
-  <link name="charger_link">
+  <!--link name="charger_link">
     <collision>
       <origin xyz="0.0 0.0 0.0" rpy="0 0 0"/>
@@ -384,25 +384,25 @@
       <xacro:Charger_Inertia />
     </inertial>
-  </link>
+  </link-->
   <!--////////////////////////////////knife_charger_joint/////////////////////////////////-->
-  <joint name="knife_charger_joint" type="fixed">
+  <!--joint name="knife_charger_joint" type="fixed">
     <origin xyz="0.065 -0.08975 0.060" rpy="0.0 0.0 0.0"/>
     <parent link="camera_mount_link"/>
     <child link="charger_link"/>
-  </joint>
+  </joint-->
     <!--0.0149 0.047621 0.110-->
  <!-- /////////////////////////////////   world   ////////////////////////////////////// -->
   <link name="ee_link"/>
   <joint name="ee_link_joint" type="fixed">
-      <origin xyz="0 -0.11575 0.20807" rpy="-1.5707 0.0 0.0"/>
+      <origin xyz="0.10125 0.0 -0.0695" rpy="0.0 0.0 1.5707"/>
       <parent link="camera_mount_link"/>
       <child link="ee_link" />
   </joint>
-  <link name="charger_ee_link"/>
-  <joint name="charger_ee_link_joint" type="fixed">
+  <!--link name="charger_ee_link"/-->
+  <!--joint name="charger_ee_link_joint" type="fixed">
       <origin xyz="0.053 0.0 0.0" rpy="${-M_PI/2} 0.0 0.0"/>
       <parent link="charger_link"/>
       <child link="charger_ee_link" />
-  </joint>
+  </joint-->
   <link name="world" />
   <joint name="world_joint" type="fixed">
@@ -424,7 +424,7 @@
      <material>Gazebo/Gray</material>
   </gazebo>
-   <gazebo reference="charger_link">
+   <!--gazebo reference="charger_link">
      <material>Gazebo/Orange</material>
-  </gazebo>
+  </gazebo-->
   <!--////////////////////////////////// Transmissions for ROS Control //////////////////////////-->
 <xacro:macro name="aubo_arm_transmission" params="joint_name">

Commit message: update new model

File: aubo_gazebo/urdf/aubo_i5.xacro (robot description, xacro)
@@ -89,11 +89,11 @@
         <origin xyz="0 0 0"
                 rpy="0 0 0"/>
-        <mass value="0.033" />
-        <inertia  ixx="1.474E-06"
-                  ixy="0.0"
-                  ixz="0.0"
-                  iyy="7.2187E-08"
-                  iyz="0"
-                  izz="1.545727E-06" />
+        <mass value="2.900" />
+        <inertia  ixx="9.262021396E-02"
+                  ixy="4.23043326E-03"
+                  ixz="5.458128035E-02"
+                  iyy="1.3936975446E-01"
+                  iyz="9.51563616E-03"
+                  izz="6.341550849E-02" />
     </xacro:macro>
     <xacro:macro name="Camera_Inertia">
@@ -107,4 +107,15 @@
                   iyz="0.0"
                   izz="0.003879257" />
+    </xacro:macro>
+    <xacro:macro name="Camera_Mount_Inertia">
+        <origin xyz="0 0 0"
+                rpy="0 0 0"/>
+        <mass value="0.63617" />
+        <inertia  ixx="2.57390373e-03"
+                  ixy="0.4E-10"
+                  ixz="-6.204366E-04"
+                  iyy="2.87452369E-03"
+                  iyz="-7.39E-09"
+                  izz="5.2167513E-04" />
     </xacro:macro>
     <!--xacro:macro name="Charger_Inertia">
@@ -317,4 +328,29 @@
   </joint>
   <!--////////////////////////////////CameraMount_Link/////////////////////////////////-->
+  <link name="knife_link" >
+    <visual>
+      <origin xyz="0.0 0.0 0.0" rpy="0 0 0"/>
+      <geometry>
+         <mesh filename="package://aubo_description/meshes/knife.dae" />
+      </geometry>
+      <material name="aluminum"/>
+    </visual>
+    <collision>
+      <origin xyz="0.0 0.0 0.0" rpy="0 0 0"/>
+      <geometry>
+         <mesh filename="package://aubo_description/meshes/knife.dae" />
+      </geometry>
+    </collision>
+    <inertial>
+      <xacro:Knife_Inertia />
+    </inertial>
+  </link>
+  <!--////////////////////////////////CameraMount_Joint/////////////////////////////////-->
+  <joint name="knife_mount_joint" type="fixed">
+    <origin xyz="0.0 0.0 0.00275" rpy="0.0 -1.5707963 0.0"/>
+    <parent link="wrist3_Link"/>
+    <child link="knife_link"/>
+  </joint>
+  <!--////////////////////////////////CameraMount_Link/////////////////////////////////-->
   <link name="camera_mount_link" >
     <visual>
@@ -332,11 +368,11 @@
     </collision>
     <inertial>
-      <xacro:Knife_Inertia />
+      <xacro:Camera_Mount_Inertia />
     </inertial>
   </link>
   <!--////////////////////////////////CameraMount_Joint/////////////////////////////////-->
   <joint name="knife_camera_mount_joint" type="fixed">
-    <origin xyz="0.0 0.0 0.005" rpy="0.0 -1.5707 -1.5707"/>
-    <parent link="wrist3_Link"/>
+    <origin xyz="0.0 0.0606 0.000" rpy="1.5707963 0.0 -1.5707963"/>
+    <parent link="wrist2_Link"/>
     <child link="camera_mount_link"/>
   </joint>
@@ -362,5 +398,5 @@
   <!--////////////////////////////////camera_joint/////////////////////////////////-->
   <joint name="camera_joint" type="fixed">
-    <origin xyz="0.02175 0.0149 -0.0185" rpy="0.0 0.0 0"/>
+    <origin xyz="-0.01 0.0825 -0.0149" rpy="-1.5707963 0.0 0"/>
     <parent link="camera_mount_link"/>
     <child link="camera_link"/>
@@ -395,6 +431,6 @@
   <link name="ee_link"/>
   <joint name="ee_link_joint" type="fixed">
-      <origin xyz="0.10125 0.0 -0.0695" rpy="0.0 0.0 1.5707"/>
-      <parent link="camera_mount_link"/>
+      <origin xyz="0.142 0.0 0.0405" rpy="0.0 1.5707963 1.5707"/>
+      <parent link="knife_link"/>
       <child link="ee_link" />
   </joint>

Commit message: new model

File: aubo_gazebo/urdf/aubo_i5.xacro (robot description, xacro)
@@ -153,4 +153,32 @@
     </collision>
   </link>
+  <link name="velodyne">
+    <visual>
+      <origin xyz="0.0 0.0 0.0"/>
+      <geometry>
+        <cylinder length="0.07" radius="0.05" />
+      </geometry>
+      <material name="gray" />
+    </visual>
+  </link>
+  <link name="imu_link">
+    <visual>
+      <origin xyz="0.0 0.0 0.0" />
+      <geometry>
+        <box size="0.04 0.02 0.01" />
+      </geometry>
+      <material name="orange" />
+    </visual>
+  </link>
+  <joint name="imu_link_joint" type="fixed">
+    <parent link="base_link" />
+    <child link="imu_link" />
+    <origin xyz="0. 0. 0." rpy="0 0 0" />
+  </joint>
+  <joint name="velodyne_joint" type="fixed">
+    <parent link="base_link" />
+    <child link="velodyne" />
+    <origin xyz="0.32 0 0.035" rpy="0 0 0" />
+  </joint>
   <!--/////////////////////////////// SHOULDER_LINK ////////////////////////////////////-->
   <link name="shoulder_Link">
@@ -339,5 +367,5 @@
       <origin xyz="0.0 0.0 0.0" rpy="0 0 0"/>
       <geometry>
-         <mesh filename="package://aubo_description/meshes/knife.dae" />
+         <mesh filename="package://aubo_description/meshes/knife.stl" />
       </geometry>
     </collision>
@@ -348,5 +376,5 @@
   <!--////////////////////////////////CameraMount_Joint/////////////////////////////////-->
   <joint name="knife_mount_joint" type="fixed">
-    <origin xyz="0.0 0.0 0.00275" rpy="0.0 -1.5707963 0.0"/>
+    <origin xyz="0.0 0.0 0.00575" rpy="0.0 -1.5707963 0.0"/>
     <parent link="wrist3_Link"/>
     <child link="knife_link"/>
@@ -373,6 +401,6 @@
   <!--////////////////////////////////CameraMount_Joint/////////////////////////////////-->
   <joint name="knife_camera_mount_joint" type="fixed">
-    <origin xyz="0.0 0.0606 0.000" rpy="1.5707963 0.0 -1.5707963"/>
-    <parent link="wrist2_Link"/>
+    <origin xyz="0.0 0.0 0.0001" rpy="0.00 0.0 0.0277"/>
+    <parent link="wrist3_Link"/>
     <child link="camera_mount_link"/>
   </joint>
@@ -398,5 +426,5 @@
   <!--////////////////////////////////camera_joint/////////////////////////////////-->
   <joint name="camera_joint" type="fixed">
-    <origin xyz="-0.01 0.0825 -0.0149" rpy="-1.5707963 0.0 0"/>
+    <origin xyz="0.01868 0.098 -0.07008" rpy="-1.5707 0.0 0"/>
     <parent link="camera_mount_link"/>
     <child link="camera_link"/>
@@ -441,10 +469,4 @@
       <child link="charger_ee_link" />
   </joint-->
-  <link name="world" />
-  <joint name="world_joint" type="fixed">
-    <parent link="world" />
-    <child link = "base_link" />
-    <origin xyz="0.0 0.0 0.0" rpy="0.0 0.0 0.0" />
-  </joint>
   <link name="virtual_camera_color_frame" />
   <joint name="virtual_camera_joint" type="fixed">

Commit message: the first full version of rubber tapping robot

File: aubo_gazebo/urdf/aubo_i5.xacro (robot description, xacro)
@@ -89,11 +89,11 @@
         <origin xyz="0 0 0"
                 rpy="0 0 0"/>
-        <mass value="0.033" />
-        <inertia  ixx="1.474E-06"
-                  ixy="0.0"
-                  ixz="0.0"
-                  iyy="7.2187E-08"
-                  iyz="0"
-                  izz="1.545727E-06" />
+        <mass value="2.900" />
+        <inertia  ixx="9.262021396E-02"
+                  ixy="4.23043326E-03"
+                  ixz="5.458128035E-02"
+                  iyy="1.3936975446E-01"
+                  iyz="9.51563616E-03"
+                  izz="6.341550849E-02" />
     </xacro:macro>
     <xacro:macro name="Camera_Inertia">
@@ -107,4 +107,15 @@
                   iyz="0.0"
                   izz="0.003879257" />
+    </xacro:macro>
+    <xacro:macro name="Camera_Mount_Inertia">
+        <origin xyz="0 0 0"
+                rpy="0 0 0"/>
+        <mass value="0.63617" />
+        <inertia  ixx="2.57390373e-03"
+                  ixy="0.4E-10"
+                  ixz="-6.204366E-04"
+                  iyy="2.87452369E-03"
+                  iyz="-7.39E-09"
+                  izz="5.2167513E-04" />
     </xacro:macro>
     <!--xacro:macro name="Charger_Inertia">
@@ -142,4 +153,32 @@
     </collision>
   </link>
+  <link name="velodyne">
+    <visual>
+      <origin xyz="0.0 0.0 0.0"/>
+      <geometry>
+        <cylinder length="0.07" radius="0.05" />
+      </geometry>
+      <material name="gray" />
+    </visual>
+  </link>
+  <link name="imu_link">
+    <visual>
+      <origin xyz="0.0 0.0 0.0" />
+      <geometry>
+        <box size="0.04 0.02 0.01" />
+      </geometry>
+      <material name="orange" />
+    </visual>
+  </link>
+  <joint name="imu_link_joint" type="fixed">
+    <parent link="base_link" />
+    <child link="imu_link" />
+    <origin xyz="0. 0. 0." rpy="0 0 0" />
+  </joint>
+  <joint name="velodyne_joint" type="fixed">
+    <parent link="base_link" />
+    <child link="velodyne" />
+    <origin xyz="0.32 0 0.035" rpy="0 0 0" />
+  </joint>
   <!--/////////////////////////////// SHOULDER_LINK ////////////////////////////////////-->
   <link name="shoulder_Link">
@@ -317,4 +356,29 @@
   </joint>
   <!--////////////////////////////////CameraMount_Link/////////////////////////////////-->
+  <link name="knife_link" >
+    <visual>
+      <origin xyz="0.0 0.0 0.0" rpy="0 0 0"/>
+      <geometry>
+         <mesh filename="package://aubo_description/meshes/knife.STL" />
+      </geometry>
+      <!--material name="aluminum"/-->
+    </visual>
+    <collision>
+      <origin xyz="0.0 0.0 0.0" rpy="0 0 0"/>
+      <geometry>
+         <mesh filename="package://aubo_description/meshes/knife.STL" />
+      </geometry>
+    </collision>
+    <inertial>
+      <xacro:Knife_Inertia />
+    </inertial>
+  </link>
+  <!--////////////////////////////////CameraMount_Joint/////////////////////////////////-->
+  <joint name="knife_mount_joint" type="fixed">
+    <origin xyz="0.0 0.0 0.00575" rpy="1.5707 0.0 3.1415"/>
+    <parent link="wrist3_Link"/>
+    <child link="knife_link"/>
+  </joint>
+  <!--////////////////////////////////CameraMount_Link/////////////////////////////////-->
   <link name="camera_mount_link" >
     <visual>
@@ -332,10 +396,10 @@
     </collision>
     <inertial>
-      <xacro:Knife_Inertia />
+      <xacro:Camera_Mount_Inertia />
     </inertial>
   </link>
   <!--////////////////////////////////CameraMount_Joint/////////////////////////////////-->
   <joint name="knife_camera_mount_joint" type="fixed">
-    <origin xyz="0.0 0.0 0.005" rpy="0.0 -1.5707 -1.5707"/>
+    <origin xyz="0.0 0.0 0.0001" rpy="0.00 0.0 0.0277"/>
     <parent link="wrist3_Link"/>
     <child link="camera_mount_link"/>
@@ -362,5 +426,5 @@
   <!--////////////////////////////////camera_joint/////////////////////////////////-->
   <joint name="camera_joint" type="fixed">
-    <origin xyz="0.02175 0.0149 -0.0185" rpy="0.0 0.0 0"/>
+    <origin xyz="0.03358 0.098 -0.05518" rpy="-1.5707 -1.5707 0"/>
     <parent link="camera_mount_link"/>
     <child link="camera_link"/>
@@ -395,6 +459,6 @@
   <link name="ee_link"/>
   <joint name="ee_link_joint" type="fixed">
-      <origin xyz="0.10125 0.0 -0.0695" rpy="0.0 0.0 1.5707"/>
-      <parent link="camera_mount_link"/>
+      <origin xyz="0.0 0.0 0.2" rpy="-1.5707 0.0 0.0"/>
+      <parent link="wrist3_Link"/>
       <child link="ee_link" />
   </joint>
@@ -405,10 +469,4 @@
       <child link="charger_ee_link" />
   </joint-->
-  <link name="world" />
-  <joint name="world_joint" type="fixed">
-    <parent link="world" />
-    <child link = "base_link" />
-    <origin xyz="0.0 0.0 0.0" rpy="0.0 0.0 0.0" />
-  </joint>
   <link name="virtual_camera_color_frame" />
   <joint name="virtual_camera_joint" type="fixed">
